Commit message: 2024.6.23 fix:improve logic

File: rm_control/rm_description/urdf/balance/chassis.urdf.xacro (robot description, xacro)
@@ -7,6 +7,6 @@
     <xacro:property name="wheel_base" value="0.4"/>
     <xacro:property name="leg_z_offset" value="-0.068374"/>
-    <xacro:macro name="chassis" >
-        <link name="base_link">
+    <xacro:macro name="chassis">
+        <link name="base_link" >
             <inertial>
                 <mass value="10.34269"/>  <!--连杆质量 -->
@@ -17,13 +17,13 @@
             <visual>
                 <origin xyz="0 0 0" rpy="0 0 0"/>
-                <!-- <geometry>
+                <geometry>
                     <mesh filename="package://rm_description/meshes/hero/base.stl" scale="0.001 .001 0.001"/>
-                </geometry> -->
+                </geometry>
             </visual>
             <collision>
                 <origin xyz="0 0 0" rpy="0 0 0"/>
-                <!-- <geometry>
+                <geometry>
                     <mesh filename="package://rm_description/meshes/hero/base.stl" scale="0.001 0.001 0.001"/>
-                </geometry> -->
+                </geometry>
             </collision>
         </link>
@@ -34,6 +34,6 @@
                             leg_y_offset="${wheel_track/2}"
                             leg_z_offset="${leg_z_offset}"
-                            mechanical_reduction="9"/>
-        <xacro:second_leg prefix="left_front" connected_to="base_link"
+                            mechanical_reduction="1"/>
+        <xacro:second_leg prefix="left_front" connected_to="left_front_first_leg"
                             pitch_offset="0"
                             leg_x_offset="${wheel_base/2}"
@@ -46,6 +46,6 @@
                             leg_y_offset="${wheel_track/2}"
                             leg_z_offset="${leg_z_offset}"
-                            mechanical_reduction="9"/>
-        <xacro:second_leg prefix="left_back" connected_to="base_link"
+                            mechanical_reduction="1"/>
+        <xacro:second_leg prefix="left_back" connected_to="left_back_first_leg"
                             pitch_offset="0"
                             leg_x_offset="${wheel_base/2}"
@@ -58,6 +58,6 @@
                             leg_y_offset="${wheel_track/2}"
                             leg_z_offset="${leg_z_offset}"
-                            mechanical_reduction="9"/>
-        <xacro:second_leg prefix="right_front" connected_to="base_link"
+                            mechanical_reduction="1"/>
+        <xacro:second_leg prefix="right_front" connected_to="right_front_first_leg"
                             pitch_offset="0"
                             leg_x_offset="${wheel_base/2}"
@@ -70,5 +70,5 @@
                             leg_y_offset="${wheel_track/2}"
                             leg_z_offset="${leg_z_offset}"
-                            mechanical_reduction="9"/>
+                            mechanical_reduction="1"/>
         <xacro:second_leg prefix="right_back" connected_to="right_back_first_leg"
                             pitch_offset="0"
@@ -76,5 +76,6 @@
                             leg_y_offset="${wheel_track/2}"
                             leg_z_offset="${leg_z_offset}"/>
-        <!-- <xacro:wheel_transmission prefix="left" mechanical_reduction="19.2032"/>
+<!--
+        <xacro:wheel_transmission prefix="left" mechanical_reduction="19.2032"/>
         <xacro:wheel_transmission prefix="right" mechanical_reduction="-19.2032"/> -->
     </xacro:macro>

Commit message: 2024.7.20 hw: dm_motor_init && lk_motor多电机力矩

File: rm_control/rm_description/urdf/balance/chassis.urdf.xacro (robot description, xacro)
@@ -1,10 +1,13 @@
 <robot xmlns:xacro="http://www.ros.org/wiki/xacro">
-    <!-- <xacro:include filename="$(find rm_description)/urdf/common/mecanum_wheel.urdf.xacro"/> -->
+    <xacro:include filename="$(find rm_description)/urdf/common/mecanum_wheel.urdf.xacro"/>
     <!-- <xacro:include filename="$(find rm_description)/urdf/common/omni_wheel.urdf.xacro"/> -->
     <xacro:include filename="$(find rm_description)/urdf/common/leg.urdf.xacro"/>
+    <!-- <xacro:include filename="$(find rm_description)/urdf/balance/reaction_wheel.urdf.xacro"/> -->
+    <!-- <xacro:include filename="$(find rm_description)/urdf/common/swerve_drive.urdf.xacro"/> -->
     <!-- https://upload.wikimedia.org/wikipedia/commons/5/52/Wheelbase_and_Track.png -->
     <xacro:property name="wheel_track" value="0.4"/>
     <xacro:property name="wheel_base" value="0.4"/>
     <xacro:property name="leg_z_offset" value="-0.068374"/>
+    <xacro:property name="wheel_offset_z" value="-0.068374"/>
     <xacro:macro name="chassis">
         <link name="base_link" >
@@ -76,7 +79,16 @@
                             leg_y_offset="${wheel_track/2}"
                             leg_z_offset="${leg_z_offset}"/>
-<!--
-        <xacro:wheel_transmission prefix="left" mechanical_reduction="19.2032"/>
-        <xacro:wheel_transmission prefix="right" mechanical_reduction="-19.2032"/> -->
+        <xacro:mecanum_wheel prefix="left" connected_to="left_front_second_leg"
+                             wheel_x_offset="${-wheel_track/2}" wheel_y_offset="${wheel_base/2}"
+                             wheel_z_offset="${wheel_offset_z}"
+                             reflect="-1" roller_type="simple"
+                             max_effort="5" max_velocity="50"/>
+        <xacro:mecanum_wheel prefix="right" connected_to="right_front_second_leg"
+                             wheel_x_offset="${-wheel_track/2}" wheel_y_offset="${-wheel_base/2}"
+                             wheel_z_offset="${wheel_offset_z}"
+                             reflect="1" roller_type="simple"
+                             max_effort="5" max_velocity="50"/>
+        <xacro:wheel_transmission prefix="left" mechanical_reduction="1.0"/>
+        <xacro:wheel_transmission prefix="right" mechanical_reduction="-1.0"/>
     </xacro:macro>
 </robot>

Commit message: 2024.9.15 加debug数据 优化转can协议

File: rm_control/rm_description/urdf/balance/chassis.urdf.xacro (robot description, xacro)
@@ -83,10 +83,10 @@
                              wheel_z_offset="${wheel_offset_z}"
                              reflect="1" roller_type="simple"
-                             max_effort="5" max_velocity="50"/>
+                             max_effort="10" max_velocity="50"/>
         <xacro:mecanum_wheel prefix="right" connected_to="right_front_second_leg"
                              wheel_x_offset="${-wheel_track/2}" wheel_y_offset="${-wheel_base/2}"
                              wheel_z_offset="${wheel_offset_z}"
                              reflect="-1" roller_type="simple"
-                             max_effort="5" max_velocity="50"/>
+                             max_effort="10" max_velocity="50"/>
         <xacro:wheel_transmission prefix="left" mechanical_reduction="1.0"/>
         <xacro:wheel_transmission prefix="right" mechanical_reduction="-1.0"/>

File: rm_control/rm_description/urdf/common/leg.urdf.xacro (robot description, xacro)
@@ -1,4 +1,4 @@
 <robot xmlns:xacro="http://www.ros.org/wiki/xacro">
-    <xacro:property name="max_effort" value="12"/>
+    <xacro:property name="max_effort" value="40"/>
     <xacro:property name="max_velocity" value="20.9333"/>
     <xacro:property name="leg_upper_limit" value="1.728"/>
